Commit message: Update robot.urdf.xacro

File: description/robot.urdf.xacro (robot description, xacro)
@@ -30,24 +30,4 @@
        </collision>
    </link>
-   <link name="lidar">
-       <inertial>
-          <mass value="0.2"/>
-          <origin xyz="0 0 0" rpy="0 0 0"/>
-          <inertia ixx="0.01" ixy="0.0" ixz="0.0" iyy="0.01" iyz="0.0" izz="0.01"/>
-       </inertial>
-       <visual>
-          <geometry>
-             <cylinder radius="0.05" length="0.05" />
-          </geometry>
-          <origin xyz="0 0 0" rpy="0 0 0"/>
-          <material name="white"/>
-       </visual>
-       <collision>
-         <geometry>
-            <box size="0.1 0.1 0.05"/>
-         </geometry>
-         <origin xyz="0 0 0" rpy="0 0 0"/>
-       </collision>
-   </link>
    <xacro:macro name="wheel_link" params="prefix">
       <link name="${prefix}_wheel">
@@ -76,9 +56,4 @@
    <xacro:wheel_link prefix="left2" />
    <xacro:wheel_link prefix="right2" />
-   <joint name="base_lidar_joint" type="fixed">
-    <parent link="base_link"/>
-    <child link="lidar"/>
-    <origin xyz="0.2 0 0.075" rpy="0 0 0"/>
-   </joint>
    <joint name="base_left_wheel_joint" type="continuous">
     <parent link="base_link"/>
@@ -105,3 +80,39 @@
       <axis xyz="0 1 0"/>
    </joint>
+   <gazebo>
+	    <plugin name="front_wheel" filename="libgazebo_ros_diff_drive.so">
+    	<!-- Wheel Information -->
+        <left_joint>base_left_wheel_joint</left_joint>
+        <right_joint>base_right_wheel_joint</right_joint>
+        <wheel_separation>0.064</wheel_separation>
+        <wheel_diameter>0.1</wheel_diameter>
+        <!-- Limit -->
+        <max_wheel_torque>200</max_wheel_torque>
+        <max_wheel_acceleration>10.0</max_wheel_acceleration>
+        <!-- Output -->
+        <odometry_frame>odom</odometry_frame>
+        <robot_base_frame>base_link</robot_base_frame>
+        <publish_odom>true</publish_odom>
+        <publish_odom_tf>true</publish_odom_tf>
+        <publish_wheel_tf>true</publish_wheel_tf>
+	</plugin>
+  	</gazebo>
+	<gazebo>
+	  <plugin name="rear_wheel" filename="libgazebo_ros_diff_drive.so">
+    	<!-- Wheel Information -->
+        <left_joint>base_left_wheel2_joint</left_joint>
+        <right_joint>base_right_wheel2_joint</right_joint>
+        <wheel_separation>0.064</wheel_separation>
+        <wheel_diameter>0.1</wheel_diameter>
+        <!-- Limit -->
+        <max_wheel_torque>200</max_wheel_torque>
+        <max_wheel_acceleration>10.0</max_wheel_acceleration>
+        <!-- Output -->
+        <odometry_frame>odom</odometry_frame>
+        <robot_base_frame>base_link</robot_base_frame>
+        <publish_odom>true</publish_odom>
+        <publish_odom_tf>true</publish_odom_tf>
+        <publish_wheel_tf>true</publish_wheel_tf>
+	  </plugin>
+</gazebo>
 </robot>

Commit message: Commit after simulating the robot with Lidar sensor using Gazebo

File: description/robot.urdf.xacro (robot description, xacro)
@@ -1,33 +1,56 @@
 <?xml version="1.0"?>
 <robot name="robot" xmlns:xacro="http://www.ros.org/wiki/xacro">
-<material name="grey">
- <color rgba="0.7 0.7 0.7 1"/>
-</material>
-<material name="green">
- <color rgba="0 0.6 0 1"/>
-</material>
-<material name="white">
-<color rgba="1 1 1 1"/>
-</material>
+   <material name="grey">
+      <color rgba="0.7 0.7 0.7 1"/>
+   </material>
+   <material name="green">
+      <color rgba="0 0.6 0 1"/>
+   </material>
+   <material name="white">
+      <color rgba="1 1 1 1"/>
+   </material>
+   <!-- Chassis -->
    <link name="base_link">
-       <inertial>
-          <mass value="5.0"/>
-          <origin xyz="0 0 0" rpy="0 0 0"/>
-          <inertia ixx="0.1" ixy="0.0" ixz="0.0" iyy="0.1" iyz="0.0" izz="0.1"/>
-       </inertial>
-       <visual>
-          <geometry>
-             <box size="0.6 0.4 0.1" />
-          </geometry>
-          <origin xyz="0 0 0" rpy="0 0 0"/>
-          <material name="green"/>
-       </visual>
-       <collision>
+      <inertial>
+         <mass value="5.0"/>
+         <origin xyz="0 0 0" rpy="0 0 0"/>
+         <inertia ixx="0.1" ixy="0.0" ixz="0.0" iyy="0.1" iyz="0.0" izz="0.1"/>
+      </inertial>
+      <visual>
          <geometry>
             <box size="0.6 0.4 0.1" />
          </geometry>
          <origin xyz="0 0 0" rpy="0 0 0"/>
-       </collision>
+         <material name="green"/>
+      </visual>
+      <collision>
+         <geometry>
+            <box size="0.6 0.4 0.1" />
+         </geometry>
+         <origin xyz="0 0 0" rpy="0 0 0"/>
+      </collision>
    </link>
+   <!-- Lidar -->
+   <link name="lidar">
+      <inertial>
+         <mass value="0.2"/>
+         <origin xyz="0 0 0" rpy="0 0 0"/>
+         <inertia ixx="0.01" ixy="0.0" ixz="0.0" iyy="0.01" iyz="0.0" izz="0.01"/>
+      </inertial>
+      <visual>
+         <geometry>
+            <cylinder radius="0.05" length="0.05" />
+         </geometry>
+         <origin xyz="0 0 0" rpy="0 0 0"/>
+         <material name="white"/>
+      </visual>
+      <collision>
+         <geometry>
+            <box size="0.1 0.1 0.05"/>
+         </geometry>
+         <origin xyz="0 0 0" rpy="0 0 0"/>
+      </collision>
+   </link>
+   <!-- Wheels -->
    <xacro:macro name="wheel_link" params="prefix">
       <link name="${prefix}_wheel">
@@ -50,5 +73,5 @@
            <origin xyz="0 0 0" rpy="1.57 0 0"/>
          </collision>
-     </link>
+      </link>
    </xacro:macro>
    <xacro:wheel_link prefix="left" />
@@ -56,9 +79,10 @@
    <xacro:wheel_link prefix="left2" />
    <xacro:wheel_link prefix="right2" />
+   <!-- Joints -->
    <joint name="base_left_wheel_joint" type="continuous">
-    <parent link="base_link"/>
-    <child link="left_wheel"/>
-    <origin xyz="-0.2 0.25 -0.1" rpy="0 0 0"/>
-    <axis xyz="0 1 0"/>
+      <parent link="base_link"/>
+      <child link="left_wheel"/>
+      <origin xyz="-0.2 0.25 -0.1" rpy="0 0 0"/>
+      <axis xyz="0 1 0"/>
    </joint>
    <joint name="base_left_wheel2_joint" type="continuous">
@@ -69,8 +93,8 @@
    </joint>
    <joint name="base_right_wheel_joint" type="continuous">
-    <parent link="base_link"/>
-    <child link="right_wheel"/>
-    <origin xyz="-0.2 -0.25 -0.1" rpy="0 0 0"/>
-    <axis xyz="0 1 0"/>
+      <parent link="base_link"/>
+      <child link="right_wheel"/>
+      <origin xyz="-0.2 -0.25 -0.1" rpy="0 0 0"/>
+      <axis xyz="0 1 0"/>
    </joint>
    <joint name="base_right_wheel2_joint" type="continuous">
@@ -80,11 +104,36 @@
       <axis xyz="0 1 0"/>
    </joint>
+   <joint name="base_lidar_joint" type="fixed">
+      <parent link="base_link"/>
+      <child link="lidar"/>
+      <origin xyz="0.2 0 0.075" rpy="0 0 0"/>
+   </joint>
+   <!-- Motor Controlling PlugIn -->
    <gazebo>
-	    <plugin name="front_wheel" filename="libgazebo_ros_diff_drive.so">
-    	<!-- Wheel Information -->
-        <left_joint>base_left_wheel_joint</left_joint>
-        <right_joint>base_right_wheel_joint</right_joint>
-        <wheel_separation>0.064</wheel_separation>
-        <wheel_diameter>0.1</wheel_diameter>
+	   <plugin name="front_wheel" filename="libgazebo_ros_diff_drive.so">
+    	   <!-- Wheel Information -->
+         <left_joint>base_left_wheel_joint</left_joint>
+         <right_joint>base_right_wheel_joint</right_joint>
+         <wheel_separation>0.064</wheel_separation>
+         <wheel_diameter>0.1</wheel_diameter>
+         <!-- Limit -->
+         <max_wheel_torque>200</max_wheel_torque>
+         <max_wheel_acceleration>10.0</max_wheel_acceleration>
+         <!-- Output -->
+         <odometry_frame>odom</odometry_frame>
+         <robot_base_frame>base_link</robot_base_frame>
+         <publish_odom>true</publish_odom>
+         <publish_odom_tf>true</publish_odom_tf>
+         <publish_wheel_tf>true</publish_wheel_tf>
+	   </plugin>
+  	</gazebo>
+   <!-- Motor Controlling PlugIn -->
+	<gazebo>
+	   <plugin name="rear_wheel" filename="libgazebo_ros_diff_drive.so">
+    	   <!-- Wheel Information -->
+         <left_joint>base_left_wheel2_joint</left_joint>
+         <right_joint>base_right_wheel2_joint</right_joint>
+         <wheel_separation>0.064</wheel_separation>
+         <wheel_diameter>0.1</wheel_diameter>
         <!-- Limit -->
         <max_wheel_torque>200</max_wheel_torque>
@@ -96,23 +145,33 @@
         <publish_odom_tf>true</publish_odom_tf>
         <publish_wheel_tf>true</publish_wheel_tf>
-	</plugin>
-  	</gazebo>
-	<gazebo>
-	  <plugin name="rear_wheel" filename="libgazebo_ros_diff_drive.so">
-    	<!-- Wheel Information -->
-        <left_joint>base_left_wheel2_joint</left_joint>
-        <right_joint>base_right_wheel2_joint</right_joint>
-        <wheel_separation>0.064</wheel_separation>
-        <wheel_diameter>0.1</wheel_diameter>
-        <!-- Limit -->
-        <max_wheel_torque>200</max_wheel_torque>
-        <max_wheel_acceleration>10.0</max_wheel_acceleration>
-        <!-- Output -->
-        <odometry_frame>odom</odometry_frame>
-        <robot_base_frame>base_link</robot_base_frame>
-        <publish_odom>true</publish_odom>
-        <publish_odom_tf>true</publish_odom_tf>
-        <publish_wheel_tf>true</publish_wheel_tf>
-	  </plugin>
-</gazebo>
+	   </plugin>
+   </gazebo>
+   <!-- Lidar PlugIn -->
+   <gazebo reference="lidar">
+      <sensor name='lidar' type='ray'>"
+         <pose relative_to='lidar'>0 0 0 0 0 0</pose>
+         <topic>lidar</topic>
+         <update_rate>10</update_rate>
+         <ray>
+            <scan>
+               <horizontal>
+                  <samples>640</samples>
+                  <resolution>1</resolution>
+                  <min_angle>-3.141592653589793238462643383279502884197</min_angle>
+                  <max_angle>3.141592653589793238462643383279502884197</max_angle>
+               </horizontal>
+            </scan>
+            <range>
+               <min>0.3</min>
+               <max>12.0</max>
+               <resolution>0.01</resolution>
+            </range>
+         </ray>
+         <always_on>1</always_on>
+         <visualize>true</visualize>
+      </sensor>
+      <plugin filename="gz-sim-sensors-system" name="gz::sim::systems::Sensors">
+         <render_engine>ogre2</render_engine>
+      </plugin>
+   </gazebo>
 </robot>

Commit message: Update robot.urdf.xacro

File: description/robot.urdf.xacro (robot description, xacro)
@@ -52,4 +52,52 @@
       </collision>
    </link>
+   <xacro:macro name="third_link" params="prefix">
+      <link name="${prefix}_third_link">
+         <inertial>
+         <mass value="1.0"/>
+         <origin xyz="0 0 0" rpy="0 0 0"/>
+         <inertia ixx="0.01" ixy="0.0" ixz="0.0" iyy="0.01" iyz="0.0" izz="0.004"/>
+      </inertial>
+      <visual>
+         <geometry>
+            <box size="0.6 0.06 0.05"/>
+         </geometry>
+         <origin xyz="0 0 0" rpy="0 0 0"/>
+         <material name="green"/>
+      </visual>
+      <collision>
+         <geometry>
+            <box size="0.6 0.06 0.05" />
+         </geometry>
+         <origin xyz="0 0 0" rpy="0 0 0"/>
+      </collision>
+      </link>
+   </xacro:macro>
+   <xacro:third_link prefix="right" />
+   <xacro:third_link prefix="left" />
+   <xacro:macro name="sec_link" params="prefix">
+      <link name="${prefix}_sec_link">
+         <inertial>
+         <mass value="0.5"/>
+         <origin xyz="0 0 0" rpy="0 0 0"/>
+         <inertia ixx="0.005" ixy="0.0" ixz="0.0" iyy="0.005" iyz="0.0" izz="0.002"/>
+      </inertial>
+      <visual>
+         <geometry>
+            <box size="0.06 0.06 0.025" />
+         </geometry>
+         <origin xyz="0 0 0" rpy="0 0 0"/>
+         <material name="green"/>
+      </visual>
+      <collision>
+         <geometry>
+            <box size="0.06 0.06 0.025" />
+         </geometry>
+         <origin xyz="0 0 0" rpy="0 0 0"/>
+      </collision>
+      </link>
+   </xacro:macro>
+   <xacro:sec_link prefix="left" />
+   <xacro:sec_link prefix="right" />
    <!-- Wheels -->
    <xacro:macro name="wheel_link" params="prefix">
@@ -80,26 +128,50 @@
    <xacro:wheel_link prefix="right2" />
    <!-- Joints -->
+   <joint name="base_left_sec_link_joint" type="fixed">
+      <parent link="base_link"/>
+      <child link="left_sec_link"/>
+      <origin xyz=" 0 0.225 0" rpy="0 0 0"/>
+      <axis xyz="0 0 0"/>
+   </joint>
+   <joint name="base_right_sec_link_joint" type="fixed">
+      <parent link="base_link"/>
+      <child link="right_sec_link"/>
+      <origin xyz=" 0 -0.225 0" rpy="0 0 0"/>
+      <axis xyz="0 0 0"/>
+   </joint>
+   <joint name="right_sec_third_link_joint" type="fixed">
+      <parent link="right_sec_link"/>
+      <child link="right_third_link"/>
+      <origin xyz=" 0 -0.06 0" rpy="0 0 0"/>
+      <axis xyz="0 0 0"/>
+   </joint>
+   <joint name="left_sec_third_link_joint" type="fixed">
+      <parent link="left_sec_link"/>
+      <child link="left_third_link"/>
+      <origin xyz=" 0 0.06 0" rpy="0 0 0"/>
+      <axis xyz="0 0 0"/>
+   </joint>
    <joint name="base_left_wheel_joint" type="continuous">
-      <parent link="base_link"/>
+      <parent link="left_third_link"/>
       <child link="left_wheel"/>
-      <origin xyz="-0.2 0.25 -0.1" rpy="0 0 0"/>
+      <origin xyz="-0.2 0.08 -0.1" rpy="0 0 0"/>
       <axis xyz="0 1 0"/>
    </joint>
    <joint name="base_left_wheel2_joint" type="continuous">
-      <parent link="base_link"/>
+      <parent link="left_third_link"/>
       <child link="left2_wheel"/>
-      <origin xyz="0.2 0.25 -0.1" rpy="0 0 0"/>
+      <origin xyz="0.2 0.08 -0.1" rpy="0 0 0"/>
       <axis xyz="0 1 0"/>
    </joint>
    <joint name="base_right_wheel_joint" type="continuous">
-      <parent link="base_link"/>
+      <parent link="right_third_link"/>
       <child link="right_wheel"/>
-      <origin xyz="-0.2 -0.25 -0.1" rpy="0 0 0"/>
+      <origin xyz="-0.2 -0.08 -0.1" rpy="0 0 0"/>
       <axis xyz="0 1 0"/>
    </joint>
    <joint name="base_right_wheel2_joint" type="continuous">
-      <parent link="base_link"/>
+      <parent link="right_third_link"/>
       <child link="right2_wheel"/>
-      <origin xyz="0.2 -0.25 -0.1" rpy="0 0 0"/>
+      <origin xyz="0.2 -0.08 -0.1" rpy="0 0 0"/>
       <axis xyz="0 1 0"/>
    </joint>
@@ -107,5 +179,5 @@
       <parent link="base_link"/>
       <child link="lidar"/>
-      <origin xyz="0.2 0 0.075" rpy="0 0 0"/>
+      <origin xyz="0.25 0 0.075" rpy="0 0 0"/>
    </joint>
    <!-- Motor Controlling PlugIn -->

Commit message: Update robot.urdf.xacro with camera plugin

File: description/robot.urdf.xacro (robot description, xacro)
@@ -10,4 +10,19 @@
       <color rgba="1 1 1 1"/>
    </material>
+   <material name="black">
+      <color rgba="0.0 0.0 0.0 1.0"/>
+    </material>
+    <material name="blue">
+      <color rgba="0.0 0.0 0.8 1.0"/>
+    </material>
+    <material name="orange">
+      <color rgba="${255/255} ${108/255} ${10/255} 1.0"/>
+    </material>
+    <material name="brown">
+      <color rgba="${222/255} ${207/255} ${195/255} 1.0"/>
+    </material>
+    <material name="red">
+      <color rgba="0.8 0.0 0.0 1.0"/>
+    </material>
    <!-- Chassis -->
    <link name="base_link">
@@ -27,4 +42,24 @@
          <geometry>
             <box size="0.6 0.4 0.1" />
+         </geometry>
+         <origin xyz="0 0 0" rpy="0 0 0"/>
+      </collision>
+   </link>
+   <link name="camera">
+      <inertial>
+         <mass value="5.0"/>
+         <origin xyz="0 0 0" rpy="0 0 0"/>
+         <inertia ixx="0.1" ixy="0.0" ixz="0.0" iyy="0.1" iyz="0.0" izz="0.1"/>
+      </inertial>
+      <visual>
+         <geometry>
+            <box size="0.05 0.05 0.05" />
+         </geometry>
+         <origin xyz="0 0 0" rpy="0 0 0"/>
+         <material name="orange"/>
+      </visual>
+      <collision>
+         <geometry>
+            <box size="0.05 0.05 0.05" />
          </geometry>
          <origin xyz="0 0 0" rpy="0 0 0"/>
@@ -181,8 +216,13 @@
       <origin xyz="0.25 0 0.075" rpy="0 0 0"/>
    </joint>
+   <joint name="base_camera_joint" type="fixed">
+      <parent link="base_link"/>
+      <child link="camera"/>
+      <origin xyz="0.325 0 0" rpy="0 0 0"/>
+   </joint>
    <!-- Motor Controlling PlugIn -->
    <gazebo>
 	   <plugin name="front_wheel" filename="libgazebo_ros_diff_drive.so">
-    	   <!-- Wheel Information -->
+    	<!-- Wheel Information -->
          <left_joint>base_left_wheel_joint</left_joint>
          <right_joint>base_right_wheel_joint</right_joint>
@@ -201,7 +241,7 @@
   	</gazebo>
    <!-- Motor Controlling PlugIn -->
-	<gazebo>
+   <gazebo>
 	   <plugin name="rear_wheel" filename="libgazebo_ros_diff_drive.so">
-    	   <!-- Wheel Information -->
+    	<!-- Wheel Information -->
          <left_joint>base_left_wheel2_joint</left_joint>
          <right_joint>base_right_wheel2_joint</right_joint>
@@ -221,4 +261,5 @@
    <!-- Lidar PlugIn -->
    <gazebo reference="lidar">
+      <material>Gazebo/Blue</material>
       <sensor name='lidar' type='ray'>"
          <pose relative_to='lidar'>0 0 0 0 0 0</pose>
@@ -247,3 +288,27 @@
       </plugin>
    </gazebo>
+   <!-- Camera PlugIn -->
+   <gazebo reference="camera">
+        <material>Gazebo/Red</material>
+        <sensor name="camera" type="camera">
+            <pose> 0 0 0 0 0 0 </pose>
+            <visualize>true</visualize>
+            <update_rate>10</update_rate>
+            <camera>
+                <horizontal_fov>1.089</horizontal_fov>
+                <image>
+                    <format>R8G8B8</format>
+                    <width>640</width>
+                    <height>480</height>
+                </image>
+                <clip>
+                    <near>0.05</near>
+                    <far>8.0</far>
+                </clip>
+            </camera>
+            <plugin name="camera_controller" filename="libgazebo_ros_camera.so">
+                <frame_name>camera</frame_name>
+            </plugin>
+        </sensor>
+    </gazebo>
 </robot>

Commit message: Update robot.urdf.xacro after fixing the error with LiDar

File: description/robot.urdf.xacro (robot description, xacro)
@@ -42,4 +42,24 @@
          <geometry>
             <box size="0.6 0.4 0.1" />
+         </geometry>
+         <origin xyz="0 0 0" rpy="0 0 0"/>
+      </collision>
+   </link>
+   <link name="imu">
+      <inertial>
+         <mass value="5.0"/>
+         <origin xyz="0 0 0" rpy="0 0 0"/>
+         <inertia ixx="0.1" ixy="0.0" ixz="0.0" iyy="0.1" iyz="0.0" izz="0.1"/>
+      </inertial>
+      <visual>
+         <geometry>
+            <box size="0.02 0.02 0.02" />
+         </geometry>
+         <origin xyz="0 0 0" rpy="0 0 0"/>
+         <material name="black"/>
+      </visual>
+      <collision>
+         <geometry>
+            <box size="0.02 0.02 0.02" />
          </geometry>
          <origin xyz="0 0 0" rpy="0 0 0"/>
@@ -220,4 +240,9 @@
       <child link="camera"/>
       <origin xyz="0.325 0 0" rpy="0 0 0"/>
+   </joint>
+   <joint name="base_imu_joint" type="fixed">
+      <parent link="base_link"/>
+      <child link="imu"/>
+      <origin xyz="0 0 -0.06" rpy="0 0 0"/>
    </joint>
    <!-- Motor Controlling PlugIn -->
@@ -261,30 +286,30 @@
    <!-- Lidar PlugIn -->
    <gazebo reference="lidar">
-      <material>Gazebo/Blue</material>
-      <sensor name='lidar' type='ray'>"
-         <pose relative_to='lidar'>0 0 0 0 0 0</pose>
-         <topic>lidar</topic>
+      <sensor name="laser" type="ray">
+         <pose>0 0 0 0 0 0</pose>
+         <visualize>true</visualize>
+         <always_on>1</always_on>
          <update_rate>10</update_rate>
          <ray>
             <scan>
                <horizontal>
-                  <samples>640</samples>
-                  <resolution>1</resolution>
-                  <min_angle>-3.141592653589793238462643383279502884197</min_angle>
-                  <max_angle>3.141592653589793238462643383279502884197</max_angle>
+                  <samples>360</samples>
+                  <min_angle>-3.14</min_angle>
+                  <max_angle>3.14</max_angle>
                </horizontal>
             </scan>
             <range>
                <min>0.3</min>
-               <max>12.0</max>
-               <resolution>0.01</resolution>
+               <max>12</max>
             </range>
          </ray>
-         <always_on>1</always_on>
-         <visualize>true</visualize>
+         <plugin name="laser_controller" filename="libgazebo_ros_ray_sensor.so">
+            <ros>
+               <argument>~/out:=scan</argument>
+            </ros>
+            <output_type>sensor_msgs/LaserScan</output_type>
+            <frame_name>lidar</frame_name>
+         </plugin>
       </sensor>
-      <plugin filename="gz-sim-sensors-system" name="gz::sim::systems::Sensors">
-         <render_engine>ogre2</render_engine>
-      </plugin>
    </gazebo>
    <!-- Camera PlugIn -->
