Commit message: Update robot.urdf.xacro with GPS and an ultrasonic sensor

File: description/robot.urdf.xacro (robot description, xacro)
@@ -46,5 +46,5 @@
       </collision>
    </link>
-   <link name="imu">
+   <link name="gps">
       <inertial>
          <mass value="5.0"/>
@@ -82,4 +82,24 @@
          <geometry>
             <box size="0.05 0.05 0.05" />
+         </geometry>
+         <origin xyz="0 0 0" rpy="0 0 0"/>
+      </collision>
+   </link>
+   <link name="ultrasonic">
+      <inertial>
+         <mass value="5.0"/>
+         <origin xyz="0 0 0" rpy="0 0 0"/>
+         <inertia ixx="0.1" ixy="0.0" ixz="0.0" iyy="0.1" iyz="0.0" izz="0.1"/>
+      </inertial>
+      <visual>
+         <geometry>
+            <box size="0.02 0.02 0.02" />
+         </geometry>
+         <origin xyz="0 0 0" rpy="0 0 0"/>
+         <material name="blue"/>
+      </visual>
+      <collision>
+         <geometry>
+            <box size="0.02 0.02 0.02" />
          </geometry>
          <origin xyz="0 0 0" rpy="0 0 0"/>
@@ -234,14 +254,19 @@
       <parent link="base_link"/>
       <child link="lidar"/>
-      <origin xyz="0.25 0 0.075" rpy="0 0 0"/>
+      <origin xyz="0.2 0 0.075" rpy="0 0 0"/>
    </joint>
    <joint name="base_camera_joint" type="fixed">
       <parent link="base_link"/>
       <child link="camera"/>
-      <origin xyz="0.325 0 0" rpy="0 0 0"/>
-   </joint>
-   <joint name="base_imu_joint" type="fixed">
-      <parent link="base_link"/>
-      <child link="imu"/>
+      <origin xyz="0.325 0 0.02" rpy="0 0 0"/>
+   </joint>
+   <joint name="base_ultrasonic_joint" type="fixed">
+      <parent link="base_link"/>
+      <child link="ultrasonic"/>
+      <origin xyz="0.325 0 -0.03" rpy="0 0 0"/>
+   </joint>
+   <joint name="base_gps_joint" type="fixed">
+      <parent link="base_link"/>
+      <child link="gps"/>
       <origin xyz="0 0 -0.06" rpy="0 0 0"/>
    </joint>
@@ -306,5 +331,5 @@
          <plugin name="laser_controller" filename="libgazebo_ros_ray_sensor.so">
             <ros>
-               <argument>~/out:=scan</argument>
+               <remapping>~/out:=scan</remapping>
             </ros>
             <output_type>sensor_msgs/LaserScan</output_type>
@@ -315,25 +340,85 @@
    <!-- Camera PlugIn -->
    <gazebo reference="camera">
-        <material>Gazebo/Red</material>
-        <sensor name="camera" type="camera">
-            <pose> 0 0 0 0 0 0 </pose>
-            <visualize>true</visualize>
-            <update_rate>10</update_rate>
-            <camera>
-                <horizontal_fov>1.089</horizontal_fov>
-                <image>
-                    <format>R8G8B8</format>
-                    <width>640</width>
-                    <height>480</height>
-                </image>
-                <clip>
-                    <near>0.05</near>
-                    <far>8.0</far>
-                </clip>
-            </camera>
-            <plugin name="camera_controller" filename="libgazebo_ros_camera.so">
-                <frame_name>camera</frame_name>
-            </plugin>
-        </sensor>
-    </gazebo>
+      <material>Gazebo/Red</material>
+      <sensor name="camera" type="camera">
+         <pose> 0 0 0 0 0 0 </pose>
+         <visualize>true</visualize>
+         <update_rate>10</update_rate>
+         <camera>
+            <horizontal_fov>1.089</horizontal_fov>
+            <image>
+               <format>R8G8B8</format>
+               <width>640</width>
+               <height>480</height>
+            </image>
+            <clip>
+               <near>0.05</near>
+               <far>8.0</far>
+            </clip>
+         </camera>
+         <plugin name="camera_controller" filename="libgazebo_ros_camera.so">
+            <frame_name>camera</frame_name>
+         </plugin>
+      </sensor>
+   </gazebo>
+    <!-- GPS PlugIn -->
+   <gazebo reference="gps">
+      <sensor name="gps_sensor" type="gps">
+         <always_on>true</always_on>
+         <update_rate>1.0</update_rate>
+         <plugin name="gps_controller" filename="libgazebo_ros_gps_sensor.so">
+            <ros>
+               <!-- <namespace>/br</namespace> -->
+               <remapping>gps_controller/out:=gps</remapping>
+            </ros>
+            <frame_name>imu</frame_name>
+         </plugin>
+      </sensor>
+      <material>Gazebo/Grey</material>
+   </gazebo>
+    <!-- Ultrasonic PlugIn -->
+   <gazebo reference="ultrasonic">
+      <sensor name="ultrasonic" type="ray">
+         <always_on>true</always_on>
+         <visualize>false</visualize>
+         <pose>0.0 0 0.0 0 0 0</pose>
+         <update_rate>50</update_rate>
+         <ray>
+            <scan>
+               <horizontal>
+                  <samples>5</samples>
+                  <resolution>1.0</resolution>
+                  <min_angle>-0.18</min_angle>
+                  <max_angle>0.18</max_angle>
+               </horizontal>
+               <vertical>
+                  <samples>5</samples>
+                  <resolution>1.0</resolution>
+                  <min_angle>-0.01</min_angle>
+                  <max_angle>0.01</max_angle>
+               </vertical>
+            </scan>
+            <range>
+               <min>0.02</min>
+               <max>8</max>
+               <resolution>0.01</resolution>
+            </range>
+            <noise>
+               <type>gaussian</type>
+               <mean>0.0</mean>
+               <stddev>0.01</stddev>
+            </noise>
+         </ray>
+         <plugin name="bytes_ultrasound" filename="libgazebo_ros_ray_sensor.so">
+            <ros>
+               <namespace>distance</namespace>
+               <remapping>~/out:=pr</remapping>
+            </ros>
+            <output_type>sensor_msgs/Range</output_type>
+            <radiation_type>ultrasound</radiation_type>
+            <frame_name>ultrasonic</frame_name>
+         </plugin>
+      </sensor>
+      <material>Gazebo/Blue</material>
+   </gazebo>
 </robot>

Commit message: Update robot.urdf.xacro with another ultrasonic sensor

File: description/robot.urdf.xacro (robot description, xacro)
@@ -87,4 +87,24 @@
    </link>
    <link name="ultrasonic">
+      <inertial>
+         <mass value="5.0"/>
+         <origin xyz="0 0 0" rpy="0 0 0"/>
+         <inertia ixx="0.1" ixy="0.0" ixz="0.0" iyy="0.1" iyz="0.0" izz="0.1"/>
+      </inertial>
+      <visual>
+         <geometry>
+            <box size="0.02 0.02 0.02" />
+         </geometry>
+         <origin xyz="0 0 0" rpy="0 0 0"/>
+         <material name="blue"/>
+      </visual>
+      <collision>
+         <geometry>
+            <box size="0.02 0.02 0.02" />
+         </geometry>
+         <origin xyz="0 0 0" rpy="0 0 0"/>
+      </collision>
+   </link>
+   <link name="ultrasonic2">
       <inertial>
          <mass value="5.0"/>
@@ -264,5 +284,10 @@
       <parent link="base_link"/>
       <child link="ultrasonic"/>
-      <origin xyz="0.325 0 -0.03" rpy="0 0 0"/>
+      <origin xyz="0.31 0 -0.03" rpy="0 0 0"/>
+   </joint>
+   <joint name="base_ultrasonic2_joint" type="fixed">
+      <parent link="base_link"/>
+      <child link="ultrasonic2"/>
+      <origin xyz="-0.31 0 -0.03" rpy="0 0 0"/>
    </joint>
    <joint name="base_gps_joint" type="fixed">
@@ -422,3 +447,47 @@
       <material>Gazebo/Blue</material>
    </gazebo>
+   <gazebo reference="ultrasonic2">
+      <sensor name="ultrasonic2" type="ray">
+         <always_on>true</always_on>
+         <visualize>false</visualize>
+         <pose>0.0 0 0.0 0 0 0</pose>
+         <update_rate>50</update_rate>
+         <ray>
+            <scan>
+               <horizontal>
+                  <samples>5</samples>
+                  <resolution>1.0</resolution>
+                  <min_angle>-0.18</min_angle>
+                  <max_angle>0.18</max_angle>
+               </horizontal>
+               <vertical>
+                  <samples>5</samples>
+                  <resolution>1.0</resolution>
+                  <min_angle>-0.01</min_angle>
+                  <max_angle>0.01</max_angle>
+               </vertical>
+            </scan>
+            <range>
+               <min>0.02</min>
+               <max>8</max>
+               <resolution>0.01</resolution>
+            </range>
+            <noise>
+               <type>gaussian</type>
+               <mean>0.0</mean>
+               <stddev>0.01</stddev>
+            </noise>
+         </ray>
+         <plugin name="bytes_ultrasound2" filename="libgazebo_ros_ray_sensor.so">
+            <ros>
+               <namespace>distance</namespace>
+               <remapping>~/out:=pr2</remapping>
+            </ros>
+            <output_type>sensor_msgs/Range</output_type>
+            <radiation_type>ultrasound</radiation_type>
+            <frame_name>ultrasonic2</frame_name>
+         </plugin>
+      </sensor>
+      <material>Gazebo/Blue</material>
+   </gazebo>
 </robot>

Commit message: Update robot.urdf.xacro with base_footprint

File: description/robot.urdf.xacro (robot description, xacro)
@@ -46,4 +46,5 @@
       </collision>
    </link>
+   <link name="base_footprint"></link>
    <link name="gps">
       <inertial>
@@ -295,4 +296,9 @@
       <child link="gps"/>
       <origin xyz="0 0 -0.06" rpy="0 0 0"/>
+   </joint>
+   <joint name="base_joint" type="fixed">
+      <parent link="base_footprint"/>
+      <child link="base_link"/>
+      <origin xyz="0 0 0.2" rpy="0 0 0"/>
    </joint>
    <!-- Motor Controlling PlugIn -->

Commit message: Commit with updated urdf.xacro file

File: description/robot.urdf.xacro (robot description, xacro)
@@ -26,7 +26,8 @@
     </material>
    <!-- Chassis -->
+   <link name="base_footprint"></link>
    <link name="base_link">
       <inertial>
-         <mass value="5.0"/>
+         <mass value="2.0"/>
          <origin xyz="0 0 0" rpy="0 0 0"/>
          <inertia ixx="0.1" ixy="0.0" ixz="0.0" iyy="0.1" iyz="0.0" izz="0.1"/>
@@ -46,5 +47,4 @@
       </collision>
    </link>
-   <link name="base_footprint"></link>
    <link name="gps">
       <inertial>
@@ -315,5 +315,5 @@
          <!-- Output -->
          <odometry_frame>odom</odometry_frame>
-         <robot_base_frame>base_link</robot_base_frame>
+         <robot_base_frame>base_footprint</robot_base_frame>
          <publish_odom>true</publish_odom>
          <publish_odom_tf>true</publish_odom_tf>
@@ -334,5 +334,5 @@
         <!-- Output -->
         <odometry_frame>odom</odometry_frame>
-        <robot_base_frame>base_link</robot_base_frame>
+        <robot_base_frame>base_footprint</robot_base_frame>
         <publish_odom>true</publish_odom>
         <publish_odom_tf>true</publish_odom_tf>

Commit message: Update robot.urdf.xacro

File: description/robot.urdf.xacro (robot description, xacro)
@@ -304,4 +304,5 @@
    <!-- Motor Controlling PlugIn -->
    <gazebo>
+      <material>Gazebo/Balck</material>
 	   <plugin name="front_wheel" filename="libgazebo_ros_diff_drive.so">
     	<!-- Wheel Information -->
